Commit message: main update, we will fix

File: data/folding-mechanism/robot.urdf (robot description, URDF)
Before this commit: robot folding-mechanism, 1 links, 0 joints
Links:
- added link back_left_base_fork, mass 0.0418822; collision mesh filename=package://assets/back_left_base_fork.stl; visual mesh filename=package://assets/back_left_base_fork.stl
- added link back_link, mass 0.372616; collision mesh filename=package://assets/back_link.stl; visual mesh filename=package://assets/back_link.stl
- added link back_link_2, mass 0.372616; collision mesh filename=package://assets/back_link.stl; visual mesh filename=package://assets/back_link.stl
- added link back_link_3, mass 0.372616; collision mesh filename=package://assets/back_link.stl; visual mesh filename=package://assets/back_link.stl
- added link back_right_axle, mass 0.0246615; collision mesh filename=package://assets/back_right_axle.stl; visual mesh filename=package://assets/back_right_axle.stl
- added link back_right_base_fork, mass 0.0418822; collision mesh filename=package://assets/back_right_base_fork.stl; visual mesh filename=package://assets/back_right_base_fork.stl
- added link base, mass 1e-09; collision mesh filename=package://assets/base.stl; collision mesh filename=package://assets/ground.stl
- added link body, mass 9.21129; collision mesh filename=package://assets/body.stl; visual mesh filename=package://assets/body.stl
- added link forearm, mass 1e-09; collision mesh filename=package://assets/forearm.stl; visual mesh filename=package://assets/forearm.stl
- added link front_axle_joint, mass 0.0246615; collision mesh filename=package://assets/front_axle_joint.stl; visual mesh filename=package://assets/front_axle_joint.stl
- added link front_bottom_link, mass 0.161703; collision mesh filename=package://assets/front_bottom_link.stl; visual mesh filename=package://assets/front_bottom_link.stl
- added link front_joint_fork, mass 0.0418822; collision mesh filename=package://assets/front_joint_fork.stl; visual mesh filename=package://assets/front_joint_fork.stl
- added link left_elbow_axle, mass 1e-09; collision mesh filename=package://assets/left_elbow_axle.stl; visual mesh filename=package://assets/left_elbow_axle.stl
- added link middle_plate, mass 0.0911859; collision mesh filename=package://assets/middle_plate.stl; visual mesh filename=package://assets/middle_plate.stl
- added link middle_plate_2, mass 0.0911859; collision mesh filename=package://assets/middle_plate.stl; visual mesh filename=package://assets/middle_plate.stl
- added link middle_plate_front_axle, mass 0.0678191; collision mesh filename=package://assets/middle_plate_front_axle.stl; visual mesh filename=package://assets/middle_plate_front_axle.stl
- added link middle_plate_rear_axle, mass 0.0647364; collision mesh filename=package://assets/middle_plate_rear_axle.stl; visual mesh filename=package://assets/middle_plate_rear_axle.stl
- added link right_elbow_axle, mass 1e-09; collision mesh filename=package://assets/right_elbow_axle.stl; visual mesh filename=package://assets/right_elbow_axle.stl
- added link right_forearm, mass 1e-09; collision mesh filename=package://assets/right_forearm.stl; visual mesh filename=package://assets/right_forearm.stl
- added link right_upper_arm, mass 1e-09; collision mesh filename=package://assets/right_upper_arm.stl; visual mesh filename=package://assets/right_upper_arm.stl
- added link top_back_link, mass 0.1376; collision mesh filename=package://assets/top_back_link.stl; visual mesh filename=package://assets/top_back_link.stl
- added link top_fork, mass 0.0424455; collision mesh filename=package://assets/top_fork.stl; visual mesh filename=package://assets/top_fork.stl
- added link top_front_axle, mass 0.0678191; collision mesh filename=package://assets/top_front_axle.stl; visual mesh filename=package://assets/top_front_axle.stl
- added link top_left_link, mass 0.1376; collision mesh filename=package://assets/top_left_link.stl; visual mesh filename=package://assets/top_left_link.stl
- added link top_left_link_2, mass 0.1376; collision mesh filename=package://assets/top_left_link.stl; visual mesh filename=package://assets/top_left_link.stl
- added link top_plate, mass 0.226762; collision mesh filename=package://assets/top_plate.stl; visual mesh filename=package://assets/top_plate.stl
- added link top_rear_axle, mass 0.0110977; collision mesh filename=package://assets/top_rear_axle.stl; visual mesh filename=package://assets/top_rear_axle.stl
- added link top_rear_axle_2, mass 0.0184961; collision mesh filename=package://assets/top_rear_axle__2.stl; visual mesh filename=package://assets/top_rear_axle__2.stl
- added link top_right_link, mass 0.1376; collision mesh filename=package://assets/top_right_link.stl; visual mesh filename=package://assets/top_right_link.stl
- added link upper_arm, mass 1e-09; collision mesh filename=package://assets/upper_arm.stl; visual mesh filename=package://assets/upper_arm.stl
Joints:
- added joint cylindrical_1: type revolute, parent top_plate, child top_rear_axle, origin xyz=0.0437042 -0.0249036 1.14867e-17 rpy=-3.14159 -5.72407e-16 0.00168445, axis 0 0 1, limit lower=-3.141592653589793 upper=3.141592653589793 effort=10 velocity=10
- added joint cylindrical_10: type revolute, parent back_left_axle, child back_left_base_fork, origin xyz=0.06 -0.0492115 0.04 rpy=-1.5708 -3.46945e-18 1.5708, axis 0 0 1, limit lower=-3.141592653589793 upper=3.141592653589793 effort=10 velocity=10
- added joint cylindrical_11: type revolute, parent front_joint_fork, child front_axle_joint, origin xyz=0.02 -2.08167e-19 -0.0175 rpy=-1.5708 -0 -1.5708, axis 0 0 1, limit lower=-3.141592653589793 upper=3.141592653589793 effort=10 velocity=10
- added joint cylindrical_12: type revolute, parent middle_plate_front_axle, child top_right_link, origin xyz=4.85723e-17 -5.55112e-17 0.045 rpy=1.71797e-22 2.0413e-21 -0.609978, axis 0 0 1, limit lower=-3.141592653589793 upper=3.141592653589793 effort=10 velocity=10
- added joint cylindrical_2: type revolute, parent top_fork, child top_rear_axle_2, origin xyz=0 -0.0255 1.76291e-17 rpy=2.44517e-20 1.92716e-17 -1.56955, axis 0 0 1, limit lower=-3.141592653589793 upper=3.141592653589793 effort=10 velocity=10
- added joint cylindrical_3: type revolute, parent top_front_axle, child top_left_link_2, origin xyz=0 -2.22045e-16 0.1 rpy=-8.58656e-16 -8.02604e-16 -7.77156e-16, axis 0 0 1, limit lower=-3.141592653589793 upper=3.141592653589793 effort=10 velocity=10
- added joint cylindrical_4: type revolute, parent top_right_link, child top_front_axle, origin xyz=-0.118333 -0.253766 0 rpy=3.14159 -0 0, axis 0 0 1, limit lower=-3.141592653589793 upper=3.141592653589793 effort=10 velocity=10
- added joint cylindrical_5: type revolute, parent middle_plate_rear_axle, child back_link_2, origin xyz=-4.16334e-17 0 0.0525 rpy=-3.14159 -8.54642e-17 -0.409867, axis 0 0 1, limit lower=-3.141592653589793 upper=3.141592653589793 effort=10 velocity=10
- added joint cylindrical_6: type revolute, parent middle_plate_rear_axle, child middle_plate_2, origin xyz=-6.93889e-17 8.32667e-17 0.0475 rpy=-3.14159 -8.71082e-17 -0.388218, axis 0 0 1, limit lower=-3.141592653589793 upper=3.141592653589793 effort=10 velocity=10
- added joint cylindrical_7: type revolute, parent middle_plate_front_axle, child middle_plate, origin xyz=6.93889e-18 0 -2.46519e-32 rpy=-3.14159 -0 6.93889e-18, axis 0 0 1, limit lower=-3.141592653589793 upper=3.141592653589793 effort=10 velocity=10
- added joint cylindrical_8: type revolute, parent middle_plate_front_axle, child top_left_link, origin xyz=1.38778e-17 0 -0.055 rpy=-3.14159 -0 6.93889e-18, axis 0 0 1, limit lower=-3.141592653589793 upper=3.141592653589793 effort=10 velocity=10
- added joint cylindrical_9: type revolute, parent back_right_base_fork, child back_right_axle, origin xyz=-0.015 1.38778e-19 -0.0175 rpy=-1.5708 -0 -1.5708, axis 0 0 1, limit lower=-3.141592653589793 upper=3.141592653589793 effort=10 velocity=10
- added joint fastened_2: type fixed, parent top_plate, child body, origin xyz=-0.000750282 -0.0269154 -4.83738e-16 rpy=-1.16242 1.5708 0, axis 0 0 1, limit effort=10 velocity=10
- added joint fastened_4: type fixed, parent base, child front_joint_fork, origin xyz=-0.04 -0.0518864 0.02 rpy=3.14159 -0 0, axis 0 0 1, limit effort=10 velocity=10
- added joint fastened_5: type fixed, parent back_left_base_fork, child base, origin xyz=7.80626e-20 0.0175 0.02 rpy=1.5708 1.5708 0, axis 0 0 1, limit effort=10 velocity=10
- added joint fastened_6: type fixed, parent base, child back_right_base_fork, origin xyz=-0.08 -1.37997e-17 -6.93889e-18 rpy=3.14159 4.27642e-50 1.2326e-32, axis 0 0 1, limit effort=10 velocity=10
- added joint revolute_1: type revolute, parent top_front_axle, child top_plate, origin xyz=8.32667e-17 -3.33067e-16 0.045 rpy=3.14159 -1.17916e-15 -0.790723, axis 0 0 1, limit lower=-3.141592653589793 upper=3.141592653589793 effort=10 velocity=10
- added joint revolute_10: type revolute, parent body, child upper_arm, origin xyz=0.21 0 -0.255 rpy=1.5708 -0 -1.5708, axis 0 0 1, limit lower=-3.141592653589793 upper=3.141592653589793 effort=10 velocity=10
- added joint revolute_11: type revolute, parent right_upper_arm, child right_elbow_axle, origin xyz=-1.11022e-16 0.2719 0.0025 rpy=-8.04804e-17 4.49397e-17 3.06249, axis 0 0 1, limit lower=-3.141592653589793 upper=3.141592653589793 effort=10 velocity=10
- added joint revolute_12: type revolute, parent right_elbow_axle, child right_forearm, origin xyz=3.1225e-17 2.77556e-16 -0.0125 rpy=-4.01109e-18 1.14234e-16 -2.39736, axis 0 0 1, limit lower=-3.141592653589793 upper=3.141592653589793 effort=10 velocity=10
- added joint revolute_13: type revolute, parent upper_arm, child left_elbow_axle, origin xyz=-0.0779642 0.260483 0.0225 rpy=-1.63547e-16 -6.95894e-17 1.99722, axis 0 0 1, limit lower=-3.141592653589793 upper=3.141592653589793 effort=10 velocity=10
- added joint revolute_14: type revolute, parent left_elbow_axle, child forearm, origin xyz=5.55112e-17 0 -0.0125 rpy=4.93038e-32 6.77927e-32 0, axis 0 0 1, limit lower=-3.141592653589793 upper=3.141592653589793 effort=10 velocity=10
- added joint revolute_2: type revolute, parent top_rear_axle, child top_fork, origin xyz=1.38778e-17 -5.55112e-17 7.85779e-32 rpy=-2.64904e-16 2.71115e-16 1.73289, axis 0 0 1, limit lower=-3.141592653589793 upper=3.141592653589793 effort=10 velocity=10
- added joint revolute_3: type revolute, parent top_rear_axle_2, child top_back_link, origin xyz=1.73472e-17 0 0 rpy=-3.14159 1.04068e-16 0.491877, axis 0 0 1, limit lower=-3.141592653589793 upper=3.141592653589793 effort=10 velocity=10
- added joint revolute_4: type revolute, parent front_bottom_link, child middle_plate_front_axle, origin xyz=0.257126 0.206849 -3.45606e-16 rpy=3.14159 9.09154e-16 -0.0530963, axis 0 0 1, limit lower=-3.141592653589793 upper=3.141592653589793 effort=10 velocity=10
- added joint revolute_5: type revolute, parent front_axle_joint, child front_bottom_link, origin xyz=2.08167e-19 6.93889e-18 -0.02 rpy=3.58771e-46 2.81666e-31 2.77209e-15, axis 0 0 1, limit lower=-3.141592653589793 upper=3.141592653589793 effort=10 velocity=10
- added joint revolute_6: type revolute, parent back_left_axle, child back_link, origin xyz=0.04 -0.0492115 0.04 rpy=-1.5708 0.101767 1.5708, axis 0 0 1, limit lower=-3.141592653589793 upper=3.141592653589793 effort=10 velocity=10
- added joint revolute_7: type revolute, parent back_right_axle, child back_link_3, origin xyz=-3.48332e-17 6.93889e-18 0.015 rpy=8.52776e-34 4.15976e-32 0.00576548, axis 0 0 1, limit lower=-3.141592653589793 upper=3.141592653589793 effort=10 velocity=10
- added joint revolute_8: type revolute, parent top_back_link, child middle_plate_rear_axle, origin xyz=0.118333 0.253766 2.46519e-32 rpy=3.14159 -0 0, axis 0 0 1, limit lower=-3.141592653589793 upper=3.141592653589793 effort=10 velocity=10
- added joint revolute_9: type revolute, parent body, child right_upper_arm, origin xyz=-0.21 -2.77556e-17 -0.255 rpy=1.5708 -0.32657 -1.5708, axis 0 0 1, limit lower=-3.141592653589793 upper=3.141592653589793 effort=10 velocity=10

Commit message: updates

File: data/folding-mechanism/robot.urdf (robot description, URDF)
Before this commit: robot folding-mechanism, 31 links, 30 joints
Links:
- removed link back_left_base_fork
- removed link back_link
- removed link back_link_2
- removed link back_link_3
- removed link back_right_axle
- removed link back_right_base_fork
- removed link base
- removed link body
- removed link forearm
- removed link front_axle_joint
- removed link front_bottom_link
- removed link front_joint_fork
- removed link left_elbow_axle
- removed link middle_plate
- removed link middle_plate_2
- removed link middle_plate_front_axle
- removed link middle_plate_rear_axle
- removed link right_elbow_axle
- removed link right_forearm
- removed link right_upper_arm
- removed link top_back_link
- removed link top_fork
- removed link top_front_axle
- removed link top_left_link
- removed link top_left_link_2
- removed link top_plate
- removed link top_rear_axle
- removed link top_rear_axle_2
- removed link top_right_link
- removed link upper_arm
Joints:
- removed joint cylindrical_1
- removed joint cylindrical_10
- removed joint cylindrical_11
- removed joint cylindrical_12
- removed joint cylindrical_2
- removed joint cylindrical_3
- removed joint cylindrical_4
- removed joint cylindrical_5
- removed joint cylindrical_6
- removed joint cylindrical_7
- removed joint cylindrical_8
- removed joint cylindrical_9
- removed joint fastened_2
- removed joint fastened_4
- removed joint fastened_5
- removed joint fastened_6
- removed joint revolute_1
- removed joint revolute_10
- removed joint revolute_11
- removed joint revolute_12
- removed joint revolute_13
- removed joint revolute_14
- removed joint revolute_2
- removed joint revolute_3
- removed joint revolute_4
- removed joint revolute_5
- removed joint revolute_6
- removed joint revolute_7
- removed joint revolute_8
- removed joint revolute_9
